Commit message: mapping wait TF with joy

File: description/lidar.xacro (robot description, xacro)
@@ -4,8 +4,9 @@
         <parent link="chassis"/>
         <child link="laser_frame"/>
-        <origin xyz="0.338 0 1.027" rpy="0 0 0"/>
+        <origin xyz="0.338 0 0.1437" rpy="0 0 0"/>
     </joint>
     <link name="laser_frame">
         <visual>
+            <origin xyz="0 0 -0.0087"/>
             <geometry>
                 <cylinder radius="0.064" length="0.036"/>

File: description/robot.urdf.xacro (robot description, xacro)
@@ -1,5 +1,6 @@
 <?xml version="1.0"?>
 <robot xmlns:xacro="http://www.ros.org/wiki/xacro"  name="robot">
-  <xacro:include filename="robot_core.xacro" />
-  <xacro:include filename="lidar.xacro" />
+  <xacro:include filename="robot_core.xacro"/>
+  <xacro:include filename="lidar.xacro"/>
+  <xacro:include filename="ros2_control.xacro" />
 </robot>

File: description/robot_core.xacro (robot description, xacro)
@@ -17,26 +17,34 @@
   <link name="base_link">
   </link>
+  <!-- base footprint link -->
+  <joint name="base_footprint_joint" type="fixed">
+        <parent link="base_link"/>
+        <child link="base_footprint"/>
+        <origin xyz="0 0 0" rpy="0 0 0"/>
+  </joint>
+  <link name="base_footprint">
+  </link>
   <!-- chassis link -->
   <joint name="chassis_joint" type="fixed">
     <parent link="base_link"/>
     <child link="chassis"/>
-    <origin xyz="-0.25 0 0"/>
+    <origin xyz="-0.25 0 0.07"/>
   </joint>
   <link name="chassis">
     <visual>
-      <origin xyz="0.25 0 0.5"/>
+      <origin xyz="0.25 0 0.0585"/>
       <geometry>
-        <box size="0.5 0.5 1"/>
+        <box size="0.5 0.5 0.117"/>
       </geometry>
       <material name="white"/>
     </visual>
     <collision>
-      <origin xyz="0.25 0 0.5"/>
+      <origin xyz="0.25 0 0.0585"/>
       <geometry>
-        <box size="0.5 0.5 1"/>
+        <box size="0.5 0.5 0.117"/>
       </geometry>
     </collision>
     <xacro:inertial_box mass="5" x="0.5" y="0.5" z="1">
-        <origin xyz="0.25 0 0.5" rpy="0 0 0"/>
+        <origin xyz="0.25 0 0.0585" rpy="0 0 0"/>
     </xacro:inertial_box>
   </link>
@@ -45,5 +53,5 @@
     <parent link="base_link"/>
     <child link="left_wheel"/>
-    <origin xyz="0 0.12 -0.035" rpy="-${pi/2} 0 0"/>
+    <origin xyz="0 0.12 0.035" rpy="-${pi/2} 0 0"/>
     <axis xyz="0 0 1"/>
   </joint>
@@ -68,5 +76,5 @@
     <parent link="base_link"/>
     <child link="right_wheel"/>
-    <origin xyz="0 -0.12 -0.035" rpy="${pi/2} 0 0"/>
+    <origin xyz="0 -0.12 0.035" rpy="${pi/2} 0 0"/>
     <axis xyz="0 0 -1"/>
   </joint>
@@ -91,5 +99,5 @@
     <parent link="base_link"/>
     <child link="caster_wheel_UL"/>
-    <origin xyz="${0.25-0.047} ${0.25-(0.059/2)} -0.035" rpy="-${pi/2} 0 0"/>
+    <origin xyz="${0.25-0.047} ${0.25-(0.059/2)} 0.035" rpy="-${pi/2} 0 0"/>
     <axis xyz="0 0 1"/>
   </joint>
@@ -114,5 +122,5 @@
     <parent link="base_link"/>
     <child link="caster_wheel_UR"/>
-    <origin xyz="${0.25-0.047} ${-0.25+(0.059/2)} -0.035" rpy="${pi/2} 0 0"/>
+    <origin xyz="${0.25-0.047} ${-0.25+(0.059/2)} 0.035" rpy="${pi/2} 0 0"/>
     <axis xyz="0 0 1"/>
   </joint>
@@ -137,5 +145,5 @@
     <parent link="base_link"/>
     <child link="caster_wheel_LL"/>
-    <origin xyz="${-0.25+0.047} ${0.25-(0.059/2)} -0.035" rpy="-${pi/2} 0 0"/>
+    <origin xyz="${-0.25+0.047} ${0.25-(0.059/2)} 0.035" rpy="-${pi/2} 0 0"/>
     <axis xyz="0 0 1"/>
   </joint>
@@ -160,5 +168,5 @@
     <parent link="base_link"/>
     <child link="caster_wheel_LR"/>
-    <origin xyz="${-0.25+0.047} ${-0.25+(0.059/2)} -0.035" rpy="${pi/2} 0 0"/>
+    <origin xyz="${-0.25+0.047} ${-0.25+(0.059/2)} 0.035" rpy="${pi/2} 0 0"/>
     <axis xyz="0 0 1"/>
   </joint>
